File: KiCad/ESP32-BMS_Ctrl/ESP32-BMS_Ctrl.kicad_pcb (KiCad board)
At the start: 2 copper layers, 125.1 x 90.2 mm, 44 parts, among them J1 Screw_Terminal_01x02, J2 Screw_Terminal_01x02, J3 Screw_Terminal_01x02, J4 Conn_01x02, J5 Conn_01x02, J6 DE9_Receptacle_MountingHoles, J7 Screw_Terminal_01x02, Q1 IRF4905PBF, Q2 IRF4905PBF, Q3 IRF4905PBF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

Commit message: Updated Main PCB to v1.2
Other:
- board text added: "ESP32-BMS_Ctrl v1.2 https://github.com/juepi"
- board text removed: "ESP32-BMS_Ctrl v1.1 https://github.com/juepi"
Changed lines of the file:
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@@
     (effects (font (size 2 2) (thickness 0.4)) (justify left bottom))
   )
-  (gr_text "ESP32-BMS_Ctrl v1.1\nhttps://github.com/juepi" (at 101.6 100.965 90) (layer "F.Cu")
+  (gr_text "ESP32-BMS_Ctrl v1.2\nhttps://github.com/juepi" (at 101.6 100.965 90) (layer "F.Cu")
     (effects (font (size 1.5 1.5) (thickness 0.3) bold) (justify left bottom))
   )
@@
   )
   (zone (net 2) (net_name "GND") (layer "B.Cu") (hatch edge 0.5)
+    (priority 6)
+    (connect_pads (clearance 0.5))
+    (min_thickness 0.25) (filled_areas_thickness no)
+    (fill yes (thermal_gap 0.5) (thermal_bridge_width 1))
+    (polygon
+      (pts
+        (xy 218.44 132.08)
+        (xy 218.44 111.76)
+        (xy 93.345 111.76)
+        (xy 93.345 132.08)
+      )
+    )
+  )
+  (zone (net 2) (net_name "GND") (layer "B.Cu") (hatch edge 0.5)
     (connect_pads (clearance 0.5))
     (min_thickness 0.25) (filled_areas_thickness no)
@@
     (polygon
       (pts
-        (xy 93.345 132.08)
+        (xy 93.345 111.76)
         (xy 93.345 50.165)
         (xy 218.44 50.165)
-        (xy 218.44 132.08)
-      )
-    )
+        (xy 218.44 111.76)
+      )
+    )

Commit message: minor updates on main PCB
Parts:
- J4, J5: footprint Connector_JST:JST_XH_B2B-XH-AM_1x02_P2.50mm_Vertical -> Connector_JST:JST_XH_B2B-XH-A_1x02_P2.50mm_Vertical
- moved Q1 2.61 mm to (111.0, 111.8)
- moved Q2 2.61 mm to (135.9, 111.8)
- moved Q3 2.61 mm to (161.3, 111.8)
- moved D1 2.31 mm to (108.5, 118.1)
- moved D2 2.31 mm to (133.3, 118.1)
- moved D3 2.31 mm to (158.8, 118.1)
- moved J1 0.70 mm to (112.4, 125.7)
- moved J2 0.70 mm to (137.2, 125.7)
- moved J3 0.70 mm to (162.6, 125.7)
- moved J7 0.70 mm to (190.5, 125.7)
Routing:
- net Net-(Q3-G): track 15.3 -> 17.9 mm
- net Net-(Q2-G): track 15.3 -> 17.9 mm
- net Net-(Q1-G): track 15.2 -> 17.8 mm
Other:
- board text added: "Antenna"
- board text added: "USB-Conn."

Commit message: OneWire working now; updated KiCad data
Connections:
- U3 pad 31: /OW-Data -> unconnected-(U3-IO39-Pad31)
- U3 pad 5: unconnected-(U3-IO4-Pad5) -> /OW-Data
Routing:
- net /OW-Data: track 33.7 -> 59.0 mm
Other:
- board text added: "ESP32-BMS_Ctrl v1.3 https://github.com/juepi"
- board text removed: "ESP32-BMS_Ctrl v1.2 https://github.com/juepi"
Changed lines of the file:
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@@
   (net 30 "unconnected-(U3-IO1-Pad2)")
   (net 31 "unconnected-(U3-IO2-Pad3)")
-  (net 32 "unconnected-(U3-IO4-Pad5)")
+  (net 32 "unconnected-(U3-IO39-Pad31)")
   (net 33 "unconnected-(U3-IO8-Pad9)")
   (net 34 "unconnected-(U3-IO9-Pad10)")
@@
     (fp_line (start 4.95 3.4) (end 4.95 -2.35)
       (stroke (width 0.1) (type solid)) (layer "F.Fab"))
-    (pad "1" thru_hole roundrect (at 0 0 180) (size 1.7 2) (drill 1) (layers "*.Cu" "*.Mask") (roundrect_rratio 0.147059)
+    (pad "1" thru_hole roundrect (at 0 0 180) (size 1.7 2) (drill 1) (layers "*.Cu" "*.Mask") (roundrect_rratio 0.1470588235)
       (net 3 "Net-(J4-Pin_1)") (pinfunction "Pin_1") (pintype "passive"))
     (pad "2" thru_hole oval (at 2.5 0 180) (size 1.7 2) (drill 1) (layers "*.Cu" "*.Mask")
@@
     (fp_line (start 4.95 3.4) (end 4.95 -2.35)
       (stroke (width 0.1) (type solid)) (layer "F.Fab"))
-    (pad "1" thru_hole roundrect (at 0 0 180) (size 1.7 2) (drill 1) (layers "*.Cu" "*.Mask") (roundrect_rratio 0.147059)
+    (pad "1" thru_hole roundrect (at 0 0 180) (size 1.7 2) (drill 1) (layers "*.Cu" "*.Mask") (roundrect_rratio 0.1470588235)
       (net 5 "Net-(J5-Pin_1)") (pinfunction "Pin_1") (pintype "passive"))
     (pad "2" thru_hole oval (at 2.5 0 180) (size 1.7 2) (drill 1) (layers "*.Cu" "*.Mask")
@@
       (net 27 "/SSR2") (pinfunction "IO3") (pintype "passive"))
     (pad "5" thru_hole circle (at 3.705 -21.455) (size 1.6 1.6) (drill 0.8) (layers "*.Cu" "*.Mask")
-      (net 32 "unconnected-(U3-IO4-Pad5)") (pinfunction "IO4") (pintype "passive"))
+      (net 8 "/OW-Data") (pinfunction "IO4") (pintype "passive"))
     (pad "6" thru_hole circle (at 1.165 -21.455) (size 1.6 1.6) (drill 0.8) (layers "*.Cu" "*.Mask")
       (net 24 "/SSR1") (pinfunction "IO5") (pintype "passive"))
@@
       (net 47 "unconnected-(U3-IO38-Pad30)") (pinfunction "IO38") (pintype "passive"))
     (pad "31" thru_hole circle (at 24.275 -26.535) (size 1.6 1.6) (drill 0.8) (layers "*.Cu" "*.Mask")
-      (net 8 "/OW-Data") (pinfunction "IO39") (pintype "passive"))
+      (net 32 "unconnected-(U3-IO39-Pad31)") (pinfunction "IO39") (pintype "passive"))
     (pad "32" thru_hole circle (at 21.735 -26.535) (size 1.6 1.6) (drill 0.8) (layers "*.Cu" "*.Mask")
       (net 48 "unconnected-(U3-IO40-Pad32)") (pinfunction "IO40") (pintype "passive"))
@@
     (effects (font (size 2 2) (thickness 0.4)) (justify left bottom))
   )
-  (gr_text "ESP32-BMS_Ctrl v1.2\nhttps://github.com/juepi" (at 101.6 100.965 90) (layer "F.Cu")
+  (gr_text "ESP32-BMS_Ctrl v1.3\nhttps://github.com/juepi" (at 101.6 100.965 90) (layer "F.Cu")
     (effects (font (size 1.5 1.5) (thickness 0.3) bold) (justify left bottom))
   )
@@
     (height -12.065)
     (orientation 1)
-    (gr_text "77,4700 mm" (at 84.56 86.36 90) (layer "Dwgs.User")
+    (gr_text "77.4700 mm" (at 84.56 86.36 90) (layer "Dwgs.User")
       (effects (font (size 1.5 1.5) (thickness 0.3)))
     )
@@
     (height -13.97)
     (orientation 0)
-    (gr_text "5,0800 mm" (at 95.885 32.505) (layer "Dwgs.User")
+    (gr_text "5.0800 mm" (at 95.885 32.505) (layer "Dwgs.User")
       (effects (font (size 1 1) (thickness 0.15)))
     )
@@
     (height -13.97)
     (orientation 0)
-    (gr_text "113,0300 mm" (at 154.94 31.855) (layer "Dwgs.User")
+    (gr_text "113.0300 mm" (at 154.94 31.855) (layer "Dwgs.User")
       (effects (font (size 1.5 1.5) (thickness 0.3)))
     )
@@
     (height 24.13)
     (orientation 1)
-    (gr_text "90,1700 mm" (at 240.77 86.995 90) (layer "Dwgs.User")
+    (gr_text "90.1700 mm" (at 240.77 86.995 90) (layer "Dwgs.User")
       (effects (font (size 1.5 1.5) (thickness 0.3)))
     )
@@
     (height -14.022966)
     (orientation 0)
-    (gr_text "6,9850 mm" (at 214.9475 32.452034) (layer "Dwgs.User")
+    (gr_text "6.9850 mm" (at 214.9475 32.452034) (layer "Dwgs.User")
       (effects (font (size 1 1) (thickness 0.15)))
     )
@@
     (height 15.24)
     (orientation 0)
-    (gr_text "125,0950 mm" (at 155.8925 145.52) (layer "Dwgs.User")
+    (gr_text "125.0950 mm" (at 155.8925 145.52) (layer "Dwgs.User")
       (effects (font (size 1.5 1.5) (thickness 0.3)))
     )
@@
     (height -12.065)
     (orientation 1)
-    (gr_text "6,9850 mm" (at 85.21 128.5875 90) (layer "Dwgs.User")
+    (gr_text "6.9850 mm" (at 85.21 128.5875 90) (layer "Dwgs.User")
       (effects (font (size 1 1) (thickness 0.15)))
     )
@@
     (height -12.065)
     (orientation 1)
-    (gr_text "5,7150 mm" (at 85.21 44.7675 90) (layer "Dwgs.User")
+    (gr_text "5.7150 mm" (at 85.21 44.7675 90) (layer "Dwgs.User")
       (effects (font (size 1 1) (thickness 0.15)))
     )
@@
   (segment (start 170.815 83.751) (end 168.841 83.751) (width 0.5) (layer "B.Cu") (net 6))
   (segment (start 168.841 83.751) (end 167.005 81.915) (width 0.5) (layer "B.Cu") (net 6))
-  (segment (start 192.44 52.105) (end 201.93 61.595) (width 0.5) (layer "B.Cu") (net 8))
-  (segment (start 189.97 52.105) (end 192.44 52.105) (width 0.5) (layer "B.Cu") (net 8))
-  (segment (start 201.93 74.495331) (end 205.424669 77.99) (width 0.5) (layer "B.Cu") (net 8))
-  (segment (start 201.93 61.595) (end 201.93 74.495331) (width 0.5) (layer "B.Cu") (net 8))
+  (segment (start 205.424669 77.99) (end 204.99 77.99) (width 0.5) (layer "F.Cu") (net 8))
+  (segment (start 191.77 50.165) (end 186.055 50.165) (width 0.5) (layer "F.Cu") (net 8))
+  (segment (start 186.055 50.165) (end 179.035 57.185) (width 0.5) (layer "F.Cu") (net 8))
+  (segment (start 179.035 57.185) (end 169.4 57.185) (width 0.5) (layer "F.Cu") (net 8))
+  (segment (start 201.295 59.69) (end 191.77 50.165) (width 0.5) (layer "F.Cu") (net 8))
+  (segment (start 204.99 77.99) (end 201.295 74.295) (width 0.5) (layer "F.Cu") (net 8))
+  (segment (start 201.295 74.295) (end 201.295 59.69) (width 0.5) (layer "F.Cu") (net 8))
   (segment (start 189.97 59.725) (end 194.345 59.725) (width 0.5) (layer "F.Cu") (net 9))
   (segment (start 194.345 59.725) (end 198.12 63.5) (width 0.5) (layer "F.Cu") (net 9))
